File: Kicad/etapa_control_final/etapa_control.sch (KiCad schematic (older format))
At the start: 50 parts, among them Q1 2N3906, Q10 2N3906, Q11 2N3904, Q12 2N7000, Q13 BS250, Q2 2N3904, Q3 2N3906, Q4 2N3904, Q5 2N3904, Q6 2N3904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

Commit message: reacomodacion
Parts:
- added J1: Conn_01x01_Male, Connector_PinHeader_1.00mm:PinHeader_1x01_P1.00mm_Vertical, symbol Connector:Conn_01x01_Male
- C1, C2, C3: footprint Capacitor_THT:CP_Axial_L11.0mm_D6.0mm_P18.00mm_Horizontal -> Capacitor_THT:C_Disc_D3.8mm_W2.6mm_P2.50mm
- R_POT_1, R_POT_2, R_POT_3, R_POT_4: footprint Potentiometer_THT:Potentiometer_ACP_CA9-V10_Vertical -> Potentiometer_THT:Potentiometer_Bourns_3296W_Vertical
- SW1, SW2, SW3: footprint Button_Switch_THT:SW_CW_GPTS203211B -> Button_Switch_THT:SW_PUSH_6mm
Connections:
- net GND: now also R_POT_2.2
- net Vout: now also J1.1 (Pin_1)
Changed lines of the file:
@@
 F 0 "C1" H 8565 2846 50  0000 L CNN
 F 1 "200n" H 8565 2755 50  0000 L CNN
-F 2 "Capacitor_THT:CP_Axial_L11.0mm_D6.0mm_P18.00mm_Horizontal" H 8488 2650 50  0001 C CNN
+F 2 "Capacitor_THT:C_Disc_D3.8mm_W2.6mm_P2.50mm" H 8488 2650 50  0001 C CNN
 F 3 "~" H 8450 2800 50  0001 C CNN
 	1    8450 2800
@@
 F 0 "R_POT_3" H 6280 8204 50  0000 R CNN
 F 1 "200K" H 6280 8295 50  0000 R CNN
-F 2 "Potentiometer_THT:Potentiometer_ACP_CA9-V10_Vertical" H 6350 8250 50  0001 C CNN
+F 2 "Potentiometer_THT:Potentiometer_Bourns_3296W_Vertical" H 6350 8250 50  0001 C CNN
 F 3 "~" H 6350 8250 50  0001 C CNN
 	1    6350 8250
@@
 F 0 "R_POT_2" V 6643 3600 50  0000 C CNN
 F 1 "50K" V 6734 3600 50  0000 C CNN
-F 2 "Potentiometer_THT:Potentiometer_ACP_CA9-V10_Vertical" H 6850 3600 50  0001 C CNN
+F 2 "Potentiometer_THT:Potentiometer_Bourns_3296W_Vertical" H 6850 3600 50  0001 C CNN
 F 3 "~" H 6850 3600 50  0001 C CNN
 	1    6850 3600
@@
 F 0 "C3" H 7115 8146 50  0000 L CNN
 F 1 "0.01u" H 7115 8055 50  0000 L CNN
-F 2 "Capacitor_THT:CP_Axial_L11.0mm_D6.0mm_P18.00mm_Horizontal" H 7038 7950 50  0001 C CNN
+F 2 "Capacitor_THT:C_Disc_D3.8mm_W2.6mm_P2.50mm" H 7038 7950 50  0001 C CNN
 F 3 "~" H 7000 8100 50  0001 C CNN
 	1    7000 8100
@@
 F 0 "SW1" H 9000 5667 50  0000 C CNN
 F 1 "SW_DIP_x01" H 9000 5576 50  0000 C CNN
-F 2 "Button_Switch_THT:SW_CW_GPTS203211B" H 9000 5400 50  0001 C CNN
+F 2 "Button_Switch_THT:SW_PUSH_6mm" H 9000 5400 50  0001 C CNN
 F 3 "~" H 9000 5400 50  0001 C CNN
 	1    9000 5400
@@
 F 0 "SW2" H 9000 7067 50  0000 C CNN
 F 1 "SW_DIP_x01" H 9000 6976 50  0000 C CNN
-F 2 "Button_Switch_THT:SW_CW_GPTS203211B" H 9000 6800 50  0001 C CNN
+F 2 "Button_Switch_THT:SW_PUSH_6mm" H 9000 6800 50  0001 C CNN
 F 3 "~" H 9000 6800 50  0001 C CNN
 	1    9000 6800
@@
 F 0 "SW3" H 9000 8217 50  0000 C CNN
 F 1 "SW_DIP_x01" H 9000 8126 50  0000 C CNN
-F 2 "Button_Switch_THT:SW_CW_GPTS203211B" H 9000 7950 50  0001 C CNN
+F 2 "Button_Switch_THT:SW_PUSH_6mm" H 9000 7950 50  0001 C CNN
 F 3 "~" H 9000 7950 50  0001 C CNN
 	1    9000 7950
@@
 F 0 "R_POT_4" V 12843 6450 50  0000 C CNN
 F 1 "20K" V 12934 6450 50  0000 C CNN
-F 2 "Potentiometer_THT:Potentiometer_ACP_CA9-V10_Vertical" H 13050 6450 50  0001 C CNN
+F 2 "Potentiometer_THT:Potentiometer_Bourns_3296W_Vertical" H 13050 6450 50  0001 C CNN
 F 3 "~" H 13050 6450 50  0001 C CNN
 	1    13050 6450
@@
 F 0 "C2" H 5365 5796 50  0000 L CNN
 F 1 "0.1u" H 5365 5705 50  0000 L CNN
-F 2 "Capacitor_THT:CP_Axial_L11.0mm_D6.0mm_P18.00mm_Horizontal" H 5288 5600 50  0001 C CNN
+F 2 "Capacitor_THT:C_Disc_D3.8mm_W2.6mm_P2.50mm" H 5288 5600 50  0001 C CNN
 F 3 "~" H 5250 5750 50  0001 C CNN
 	1    5250 5750
@@
 F 0 "R_POT_1" V 4693 1500 50  0000 C CNN
 F 1 "500K" V 4784 1500 50  0000 C CNN
-F 2 "Potentiometer_THT:Potentiometer_ACP_CA9-V10_Vertical" H 4900 1500 50  0001 C CNN
+F 2 "Potentiometer_THT:Potentiometer_Bourns_3296W_Vertical" H 4900 1500 50  0001 C CNN
 F 3 "~" H 4900 1500 50  0001 C CNN
 	1    4900 1500
@@
 Wire Wire Line
 	7600 2000 7600 2050
+$Comp
+L Connector:Conn_01x01_Male J1
+U 1 1 5F0BF73C
+P 13550 6800
+F 0 "J1" V 13612 6844 50  0000 L CNN
+F 1 "Conn_01x01_Male" V 13703 6844 50  0000 L CNN
+F 2 "Connector_PinHeader_1.00mm:PinHeader_1x01_P1.00mm_Vertical" H 13550 6800 50  0001 C CNN
+F 3 "~" H 13550 6800 50  0001 C CNN
+	1    13550 6800
+	0    1    1    0
+$EndComp
+$Comp
+L power:GND #PWR0101
+U 1 1 5F0C423D
+P 6850 3750
+F 0 "#PWR0101" H 6850 3500 50  0001 C CNN
+F 1 "GND" H 6855 3577 50  0000 C CNN
+F 2 "" H 6850 3750 50  0001 C CNN
+F 3 "" H 6850 3750 50  0001 C CNN
+	1    6850 3750
+	1    0    0    -1
+$EndComp
 $EndSCHEMATC
