File: Kicad/etapa_control_final/etapa_control_final.kicad_pcb (KiCad board)
At the start: 4 copper layers, 49 parts, among them Q1 2N3906, Q10 2N3906, Q11 2N3904, Q12 2N7000, Q13 BS250, Q2 2N3904, Q3 2N3906, Q4 2N3904, Q5 2N3904, Q6 2N3904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

Commit message: reacomodacion
Parts:
- added J1: Conn_01x01_Male, Connector_PinHeader_1.00mm:PinHeader_1x01_P1.00mm_Vertical, F.Cu at (136.5, 66.0)
- added SW2: SW_DIP_x01, Button_Switch_THT:SW_PUSH_6mm, F.Cu at (117.5, 91.4)
- C1, C2, C3: footprint Capacitor_THT:CP_Axial_L11.0mm_D6.0mm_P18.00mm_Horizontal -> Capacitor_THT:C_Disc_D3.8mm_W2.6mm_P2.50mm
- R_POT_1, R_POT_2, R_POT_3, R_POT_4: footprint Potentiometer_THT:Potentiometer_ACP_CA9-V10_Vertical -> Potentiometer_THT:Potentiometer_Bourns_3296W_Vertical
- SW1, SW3: footprint Button_Switch_THT:SW_CW_GPTS203211B -> Button_Switch_THT:SW_PUSH_6mm
- moved Q9 54.7 mm to (81.3, 41.9), turned to 0 degrees
- moved R10 50.4 mm to (86.4, 58.4), turned to 270 degrees
- moved Q8 45.1 mm to (86.4, 54.6), turned to 90 degrees
- moved C2 44.6 mm to (107.3, 60.3)
- moved R23 44.0 mm to (120.0, 69.8)
- moved R_POT_1 43.2 mm to (78.7, 52.1), turned to 270 degrees
- moved Q11 43.2 mm to (94.0, 49.5)
- moved R_POT_4 42.0 mm to (128.9, 63.5), turned to 90 degrees
- moved R8 41.9 mm to (87.6, 41.9), turned to 180 degrees
- moved C3 41.0 mm to (108.6, 64.1), turned to 180 degrees
- moved U7 39.6 mm to (114.3, 68.6)
- moved R13 38.9 mm to (110.5, 76.8), turned to 0 degrees
- moved R19 36.9 mm to (123.2, 77.5)
- moved R15 36.8 mm to (106.7, 76.8), turned to 180 degrees
- moved Q12 36.4 mm to (96.5, 59.7)
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Connections:
- R11 pad 1: Net-(R11-Pad1) -> Net-(Q10-Pad1)
- R_POT_2 pad 2: Net-(R_POT_2-Pad2) -> GND
Routing:
- net GND: track 22.9 -> 156.5 mm, vias 5 -> 4
- net Net-(C2-Pad1): track 101.5 -> 43.5 mm, vias 0 -> 2
- net Net-(C1-Pad1): track 96.0 -> 50.4 mm
- net -5V: track 62.2 -> 26.9 mm, vias 0 -> 2
- net Net-(Q11-Pad2): track 52.5 -> 22.5 mm
- net Net-(R19-Pad2): track 41.4 -> 17.6 mm
- net Net-(Q10-Pad2): track 48.9 -> 26.0 mm
- net +15V: track 46.1 -> 68.2 mm, vias 6 -> 2
- net +5V: track 7.38 -> 27.6 mm
- net Net-(Q11-Pad1): track 23.0 -> 4.66 mm
- net Net-(R25-Pad2): track 6.61 -> 22.3 mm
- net Net-(R13-Pad2): track 6.74 -> 22.1 mm
- net Net-(R_POT_3-Pad2): track 30.7 -> 16.9 mm, vias 0 -> 1
- net Net-(Q1-Pad2): track 25.4 -> 12.7 mm
- net Vout: track 8.81 -> 20.3 mm
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- removed copper zone on +15, net +15V
- removed copper zone on +5, net +5V
- removed copper zone on B.Cu, net GND
Other:
- copper layers 4 -> 2
