File: Kicad/EtapaPotencia/EtapaPotencia/EtapaPotencia.sch (KiCad schematic (older format))
At the start: 65 parts, among them IC1 IRF630, IC2 IRF630, J1 Conn_01x01_Male, Q1 BC547, Q2 BC557, Q3 BC557, U1 TL082, U2 TL082, U3 TL082, U4 LM393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

Commit message: pcb
Parts:
- C1, C10, C2, C3, C7, C8: footprint (none) -> Capacitor_SMD:C_0805_2012Metric
- C11, C6: footprint (none) -> Capacitor_SMD:C_0603_1608Metric
- C20, C9: footprint (none) -> Capacitor_THT:C_Disc_D8.0mm_W5.0mm_P5.00mm
- Ct1: footprint (none) -> Capacitor_THT:C_Disc_D8.0mm_W2.5mm_P5.00mm
- J1: footprint (none) -> Connector_PinHeader_1.00mm:PinHeader_1x01_P1.00mm_Vertical
- L1: footprint (none) -> Ferrite_THT:LairdTech_28C0236-0JW-10
- U1: footprint Package_TO_SOT_THT:TO-5-2 -> Package_DIP:DIP-8_W10.16mm
- U2, U3, U4: footprint (none) -> Package_DIP:DIP-8_W10.16mm
Changed lines of the file:
@@
 F 0 "J1" V 812 2994 50  0000 L CNN
 F 1 "Conn_01x01_Male" V 903 2994 50  0000 L CNN
-F 2 "" H 750 2950 50  0001 C CNN
+F 2 "Connector_PinHeader_1.00mm:PinHeader_1x01_P1.00mm_Vertical" H 750 2950 50  0001 C CNN
 F 3 "~" H 750 2950 50  0001 C CNN
 	1    750  2950
@@
 F 0 "U1" H 1800 2767 50  0000 C CNN
 F 1 "TL082" H 1800 2676 50  0000 C CNN
-F 2 "Package_TO_SOT_THT:TO-5-2" H 1800 2400 50  0001 C CNN
+F 2 "Package_DIP:DIP-8_W10.16mm" H 1800 2400 50  0001 C CNN
 F 3 "http://www.ti.com/lit/ds/symlink/tl081.pdf" H 1800 2400 50  0001 C CNN
 	1    1800 2400
@@
 F 0 "U1" H 858 4596 50  0000 L CNN
 F 1 "TL082" H 858 4505 50  0000 L CNN
-F 2 "Package_TO_SOT_THT:TO-5-2" H 900 4550 50  0001 C CNN
+F 2 "Package_DIP:DIP-8_W10.16mm" H 900 4550 50  0001 C CNN
 F 3 "http://www.ti.com/lit/ds/symlink/tl081.pdf" H 900 4550 50  0001 C CNN
 	3    900  4550
@@
 F 0 "U2" H 3100 3967 50  0000 C CNN
 F 1 "TL082" H 3100 3876 50  0000 C CNN
-F 2 "" H 3100 3600 50  0001 C CNN
+F 2 "Package_DIP:DIP-8_W10.16mm" H 3100 3600 50  0001 C CNN
 F 3 "http://www.ti.com/lit/ds/symlink/tl081.pdf" H 3100 3600 50  0001 C CNN
 	2    3100 3600
@@
 F 0 "C9" V 2898 4500 50  0000 C CNN
 F 1 "10p" V 2989 4500 50  0000 C CNN
-F 2 "" H 3188 4350 50  0001 C CNN
+F 2 "Capacitor_THT:C_Disc_D8.0mm_W5.0mm_P5.00mm" H 3188 4350 50  0001 C CNN
 F 3 "~" H 3150 4500 50  0001 C CNN
 	1    3150 4500
@@
 F 0 "C8" H 3935 1604 50  0000 R CNN
 F 1 "1n" H 3935 1695 50  0000 R CNN
-F 2 "" H 4088 1500 50  0001 C CNN
+F 2 "Capacitor_SMD:C_0805_2012Metric" H 4088 1500 50  0001 C CNN
 F 3 "~" H 4050 1650 50  0001 C CNN
 	1    4050 1650
@@
 F 0 "C10" V 4052 2000 50  0000 C CNN
 F 1 "1n" V 3961 2000 50  0000 C CNN
-F 2 "" H 3838 1850 50  0001 C CNN
+F 2 "Capacitor_SMD:C_0805_2012Metric" H 3838 1850 50  0001 C CNN
 F 3 "~" H 3800 2000 50  0001 C CNN
 	1    3800 2000
@@
 F 0 "U4" H 4550 3333 50  0000 C CNN
 F 1 "LM393" H 4550 3424 50  0000 C CNN
-F 2 "" H 4550 3700 50  0001 C CNN
+F 2 "Package_DIP:DIP-8_W10.16mm" H 4550 3700 50  0001 C CNN
 F 3 "http://www.ti.com/lit/ds/symlink/lm393-n.pdf" H 4550 3700 50  0001 C CNN
 	1    4550 3700
@@
 F 0 "C20" H 3835 6854 50  0000 R CNN
 F 1 "0.5n" H 3835 6945 50  0000 R CNN
-F 2 "" H 3988 6750 50  0001 C CNN
+F 2 "Capacitor_THT:C_Disc_D8.0mm_W5.0mm_P5.00mm" H 3988 6750 50  0001 C CNN
 F 3 "~" H 3950 6900 50  0001 C CNN
 	1    3950 6900
@@
 F 0 "Ct1" H 4735 4204 50  0000 R CNN
 F 1 "10p" H 4735 4295 50  0000 R CNN
-F 2 "" H 4888 4100 50  0001 C CNN
+F 2 "Capacitor_THT:C_Disc_D8.0mm_W2.5mm_P5.00mm" H 4888 4100 50  0001 C CNN
 F 3 "~" H 4850 4250 50  0001 C CNN
 	1    4850 4250
@@
 F 0 "C3" H 6635 4454 50  0000 R CNN
 F 1 "30n" H 6635 4545 50  0000 R CNN
-F 2 "" H 6788 4350 50  0001 C CNN
+F 2 "Capacitor_SMD:C_0805_2012Metric" H 6788 4350 50  0001 C CNN
 F 3 "~" H 6750 4500 50  0001 C CNN
 	1    6750 4500
@@
 F 0 "C2" H 6535 3804 50  0000 R CNN
 F 1 "22n" H 6535 3895 50  0000 R CNN
-F 2 "" H 6688 3700 50  0001 C CNN
+F 2 "Capacitor_SMD:C_0805_2012Metric" H 6688 3700 50  0001 C CNN
 F 3 "~" H 6650 3850 50  0001 C CNN
 	1    6650 3850
@@
 F 0 "U2" H 908 6046 50  0000 L CNN
 F 1 "TL082" H 908 5955 50  0000 L CNN
-F 2 "" H 950 6000 50  0001 C CNN
+F 2 "Package_DIP:DIP-8_W10.16mm" H 950 6000 50  0001 C CNN
 F 3 "http://www.ti.com/lit/ds/symlink/tl081.pdf" H 950 6000 50  0001 C CNN
 	3    950  6000
@@
 F 0 "U1" H 4400 5783 50  0000 C CNN
 F 1 "TL082" H 4400 5874 50  0000 C CNN
-F 2 "Package_TO_SOT_THT:TO-5-2" H 4400 6150 50  0001 C CNN
+F 2 "Package_DIP:DIP-8_W10.16mm" H 4400 6150 50  0001 C CNN
 F 3 "http://www.ti.com/lit/ds/symlink/tl081.pdf" H 4400 6150 50  0001 C CNN
 	2    4400 6150
@@
 F 0 "U2" H 2500 5883 50  0000 C CNN
 F 1 "TL082" H 2500 5974 50  0000 C CNN
-F 2 "" H 2500 6250 50  0001 C CNN
+F 2 "Package_DIP:DIP-8_W10.16mm" H 2500 6250 50  0001 C CNN
 F 3 "http://www.ti.com/lit/ds/symlink/tl081.pdf" H 2500 6250 50  0001 C CNN
 	1    2500 6250
@@
 F 0 "L1" V 9740 4200 50  0000 C CNN
 F 1 "250u" V 9649 4200 50  0000 C CNN
-F 2 "" H 9550 4200 50  0001 C CNN
+F 2 "Ferrite_THT:LairdTech_28C0236-0JW-10" H 9550 4200 50  0001 C CNN
 F 3 "~" H 9550 4200 50  0001 C CNN
 	1    9550 4200
@@
 F 0 "C1" H 10015 4396 50  0000 L CNN
 F 1 "1u" H 10015 4305 50  0000 L CNN
-F 2 "" H 9938 4200 50  0001 C CNN
+F 2 "Capacitor_SMD:C_0805_2012Metric" H 9938 4200 50  0001 C CNN
 F 3 "~" H 9900 4350 50  0001 C CNN
 	1    9900 4350
@@
 F 0 "C6" H 10715 4396 50  0000 L CNN
 F 1 "10u" H 10715 4305 50  0000 L CNN
-F 2 "" H 10638 4200 50  0001 C CNN
+F 2 "Capacitor_SMD:C_0603_1608Metric" H 10638 4200 50  0001 C CNN
 F 3 "~" H 10600 4350 50  0001 C CNN
 	1    10600 4350
@@
 F 0 "U3" H 7200 2767 50  0000 C CNN
 F 1 "TL082" H 7200 2676 50  0000 C CNN
-F 2 "" H 7200 2400 50  0001 C CNN
+F 2 "Package_DIP:DIP-8_W10.16mm" H 7200 2400 50  0001 C CNN
 F 3 "http://www.ti.com/lit/ds/symlink/tl081.pdf" H 7200 2400 50  0001 C CNN
 	1    7200 2400
@@
 F 0 "U3" H 1608 5046 50  0000 L CNN
 F 1 "TL082" H 1608 4955 50  0000 L CNN
-F 2 "" H 1650 5000 50  0001 C CNN
+F 2 "Package_DIP:DIP-8_W10.16mm" H 1650 5000 50  0001 C CNN
 F 3 "http://www.ti.com/lit/ds/symlink/tl081.pdf" H 1650 5000 50  0001 C CNN
 	3    1650 5000
@@
 F 0 "C11" H 8785 2054 50  0000 R CNN
 F 1 "100n" H 8785 2145 50  0000 R CNN
-F 2 "" H 8938 1950 50  0001 C CNN
+F 2 "Capacitor_SMD:C_0603_1608Metric" H 8938 1950 50  0001 C CNN
 F 3 "~" H 8900 2100 50  0001 C CNN
 	1    8900 2100
@@
 F 0 "C7" V 3098 4900 50  0000 C CNN
 F 1 "100p" V 3189 4900 50  0000 C CNN
-F 2 "" H 3388 4750 50  0001 C CNN
+F 2 "Capacitor_SMD:C_0805_2012Metric" H 3388 4750 50  0001 C CNN
 F 3 "~" H 3350 4900 50  0001 C CNN
 	1    3350 4900
