File: Kicad/Etapa_potencia_funcionamiento_pcb/EtapaPotencia/EtapaPotencia.sch (KiCad schematic (older format))
At the start: 65 parts, among them IC1 IRF630, IC2 IRF630, J1 Conn_01x01_Male, Q1 BC547, Q2 BC557, Q3 BC557, U1 TL082, U2 TL082, U3 TL082, U4 LM393, U5 IRS20957S

Commit message: Actualizacion PCB
Falta acomodar el GND y ver los Loops
Parts:
- removed U1, U3: TL082, Package_DIP:DIP-8_W10.16mm, symbol Amplifier_Operational:TL082
- added U1: TL084, Package_DIP:DIP-14_W10.16mm, symbol Amplifier_Operational:TL084
- added unit 3 of U4
- D1, D2, D3: symbol eec:MUR460 -> EtapaPotencia-rescue:MUR460-eec
Connections:
- net +12V: now also U1.4 (V+), U4.4 (V-)
- net -5V: now also U1.11 (V-), U4.8 (V+)
- net GND: now also U1.3 (+), U1.5 (+)
- net at R8.1, R9.2: now also U1.2 (-)
- net at R19.2, R9.1: now also U1.1
- net at C10.1, C11.1, C9.2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: now also U1.6 (-)
- net at C7.1, C9.1, R11.2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: now also U1.7
- net at R12.2, R13.1, R14.2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: now also U1.10 (+), U1.9 (-)
- net at D4.1 (K), Q2.2 (B), R16.1: now also U1.8
Changed lines of the file:
@@
-$EndComp
-$Comp
-L Amplifier_Operational:TL082 U1
-U 1 1 5F18E47D
-P 1800 2400
-F 0 "U1" H 1800 2767 50  0000 C CNN
-F 1 "TL082" H 1800 2676 50  0000 C CNN
-F 2 "Package_DIP:DIP-8_W10.16mm" H 1800 2400 50  0001 C CNN
-F 3 "http://www.ti.com/lit/ds/symlink/tl081.pdf" H 1800 2400 50  0001 C CNN
-	1    1800 2400
-	1    0    0    -1
-$EndComp
-$Comp
-L Amplifier_Operational:TL082 U1
-U 3 1 5F193261
-P 900 4550
-F 0 "U1" H 858 4596 50  0000 L CNN
-F 1 "TL082" H 858 4505 50  0000 L CNN
-F 2 "Package_DIP:DIP-8_W10.16mm" H 900 4550 50  0001 C CNN
-F 3 "http://www.ti.com/lit/ds/symlink/tl081.pdf" H 900 4550 50  0001 C CNN
-	3    900  4550
-	1    0    0    -1
-$EndComp
-$Comp
-L Amplifier_Operational:TL082 U1
-U 2 1 5F1AD760
-P 3100 3600
-F 0 "U1" H 3100 3967 50  0000 C CNN
-F 1 "TL082" H 3100 3876 50  0000 C CNN
-F 2 "Package_DIP:DIP-8_W10.16mm" H 3100 3600 50  0001 C CNN
-F 3 "http://www.ti.com/lit/ds/symlink/tl081.pdf" H 3100 3600 50  0001 C CNN
-	2    3100 3600
-	1    0    0    -1
 $EndComp
 $Comp
@@
 	1    0    0    1
 $EndComp
-$Comp
-L Amplifier_Operational:TL082 U2
-U 1 1 5F1CA186
-P 2500 6250
-F 0 "U2" H 2500 5883 50  0000 C CNN
-F 1 "TL082" H 2500 5974 50  0000 C CNN
-F 2 "Package_DIP:DIP-8_W10.16mm" H 2500 6250 50  0001 C CNN
-F 3 "http://www.ti.com/lit/ds/symlink/tl081.pdf" H 2500 6250 50  0001 C CNN
-	1    2500 6250
-	1    0    0    1
-$EndComp
 Wire Wire Line
 	4700 6150 4850 6150
@@
 $EndComp
 $Comp
-L power:+12V #PWR01
-U 1 1 5F270AF0
-P 800 4250
-F 0 "#PWR01" H 800 4100 50  0001 C CNN
-F 1 "+12V" H 815 4423 50  0000 C CNN
-F 2 "" H 800 4250 50  0001 C CNN
-F 3 "" H 800 4250 50  0001 C CNN
-	1    800  4250
-	1    0    0    -1
-$EndComp
-$Comp
 L power:+12V #PWR03
 U 1 1 5F27177E
@@
 	1    850  5700
 	1    0    0    -1
-$EndComp
-$Comp
-L power:-5V #PWR02
-U 1 1 5F2754A6
-P 800 4850
-F 0 "#PWR02" H 800 4950 50  0001 C CNN
-F 1 "-5V" H 815 5023 50  0000 C CNN
-F 2 "" H 800 4850 50  0001 C CNN
-F 3 "" H 800 4850 50  0001 C CNN
-	1    800  4850
-	-1   0    0    1
 $EndComp
 $Comp
@@
 $EndComp
 $Comp
-L Amplifier_Operational:TL082 U3
-U 1 1 5F2BF17B
-P 7200 2400
-F 0 "U3" H 7200 2767 50  0000 C CNN
-F 1 "TL082" H 7200 2676 50  0000 C CNN
-F 2 "Package_DIP:DIP-8_W10.16mm" H 7200 2400 50  0001 C CNN
-F 3 "http://www.ti.com/lit/ds/symlink/tl081.pdf" H 7200 2400 50  0001 C CNN
-	1    7200 2400
-	1    0    0    -1
-$EndComp
-$Comp
-L Amplifier_Operational:TL082 U3
-U 3 1 5F2C4D52
-P 1650 5000
-F 0 "U3" H 1608 5046 50  0000 L CNN
-F 1 "TL082" H 1608 4955 50  0000 L CNN
-F 2 "Package_DIP:DIP-8_W10.16mm" H 1650 5000 50  0001 C CNN
-F 3 "http://www.ti.com/lit/ds/symlink/tl081.pdf" H 1650 5000 50  0001 C CNN
-	3    1650 5000
-	1    0    0    -1
-$EndComp
-$Comp
 L power:+12V #PWR06
 U 1 1 5F2C78F5
-P 1550 4700
-F 0 "#PWR06" H 1550 4550 50  0001 C CNN
-F 1 "+12V" H 1565 4873 50  0000 C CNN
-F 2 "" H 1550 4700 50  0001 C CNN
-F 3 "" H 1550 4700 50  0001 C CNN
-	1    1550 4700
+P 900 4600
+F 0 "#PWR06" H 900 4450 50  0001 C CNN
+F 1 "+12V" H 915 4773 50  0000 C CNN
+F 2 "" H 900 4600 50  0001 C CNN
+F 3 "" H 900 4600 50  0001 C CNN
+	1    900  4600
 	1    0    0    -1
 $EndComp
@@
 L power:-5V #PWR07
 U 1 1 5F2C80C1
-P 1550 5300
-F 0 "#PWR07" H 1550 5400 50  0001 C CNN
-F 1 "-5V" H 1565 5473 50  0000 C CNN
-F 2 "" H 1550 5300 50  0001 C CNN
-F 3 "" H 1550 5300 50  0001 C CNN
-	1    1550 5300
+P 900 5200
+F 0 "#PWR07" H 900 5300 50  0001 C CNN
+F 1 "-5V" H 915 5373 50  0000 C CNN
+F 2 "" H 900 5200 50  0001 C CNN
+F 3 "" H 900 5200 50  0001 C CNN
+	1    900  5200
 	-1   0    0    1
 $EndComp
@@
 Wire Wire Line
 	5650 2400 6900 2400
-Wire Wire Line
-	6900 2400 6900 2500
 Connection ~ 5650 2400
 Wire Wire Line
 	5650 2400 5650 2450
 Wire Wire Line
-	6900 2500 6900 2700
-Wire Wire Line
 	6900 2700 7050 2700
 Wire Wire Line
@@
 Wire Wire Line
 	7350 2700 7500 2700
-Connection ~ 6900 2500
 $Comp
 L power:GND #PWR018
@@
 	9200 3300 9200 3600
 $Comp
-L eec:MUR460 D3
+L EtapaPotencia-rescue:MUR460-eec D3
 U 1 1 5F21FAEE
 P 9200 4800
@@
 $EndComp
 $Comp
-L eec:MUR460 D2
+L EtapaPotencia-rescue:MUR460-eec D2
 U 1 1 5F220C6E
 P 9200 3900
@@
 $EndComp
 $Comp
-L eec:MUR460 D1
+L EtapaPotencia-rescue:MUR460-eec D1
 U 1 1 5F2217EB
 P 7250 4300
@@
 	0    -1   -1   0
 $EndComp
+$Comp
+L Comparator:LM393 U4
+U 3 1 5F1A3B33
+P 950 7150
+F 0 "U4" H 950 6783 50  0000 C CNN
+F 1 "LM393" H 950 6874 50  0000 C CNN
+F 2 "Package_DIP:DIP-8_W10.16mm" H 950 7150 50  0001 C CNN
+F 3 "http://www.ti.com/lit/ds/symlink/lm393-n.pdf" H 950 7150 50  0001 C CNN
+	3    950  7150
+	1    0    0    1
+$EndComp
+$Comp
+L power:-5V #PWR028
+U 1 1 5F1A58AA
+P 850 7450
+F 0 "#PWR028" H 850 7550 50  0001 C CNN
+F 1 "-5V" H 865 7623 50  0000 C CNN
+F 2 "" H 850 7450 50  0001 C CNN
+F 3 "" H 850 7450 50  0001 C CNN
+	1    850  7450
+	-1   0    0    1
+$EndComp
+$Comp
+L power:+12V #PWR027
+U 1 1 5F1A5C95
+P 850 6850
+F 0 "#PWR027" H 850 6700 50  0001 C CNN
+F 1 "+12V" H 865 7023 50  0000 C CNN
+F 2 "" H 850 6850 50  0001 C CNN
+F 3 "" H 850 6850 50  0001 C CNN
+	1    850  6850
+	1    0    0    -1
+$EndComp
+$Comp
+L Amplifier_Operational:TL084 U1
+U 1 1 5F1AAD94
+P 1800 2400
+F 0 "U1" H 1800 2767 50  0000 C CNN
+F 1 "TL084" H 1800 2676 50  0000 C CNN
+F 2 "Package_DIP:DIP-14_W10.16mm" H 1750 2500 50  0001 C CNN
+F 3 "http://www.ti.com/lit/ds/symlink/tl081.pdf" H 1850 2600 50  0001 C CNN
+	1    1800 2400
+	1    0    0    -1
+$EndComp
+$Comp
+L Amplifier_Operational:TL084 U1
+U 2 1 5F1ADA5E
+P 3100 3600
+F 0 "U1" H 3100 3967 50  0000 C CNN
+F 1 "TL084" H 3100 3876 50  0000 C CNN
+F 2 "Package_DIP:DIP-14_W10.16mm" H 3050 3700 50  0001 C CNN
+F 3 "http://www.ti.com/lit/ds/symlink/tl081.pdf" H 3150 3800 50  0001 C CNN
+	2    3100 3600
+	1    0    0    -1
+$EndComp
+Wire Wire Line
+	6900 2400 6900 2500
+$Comp
+L Amplifier_Operational:TL084 U1
+U 3 1 5F1AF993
+P 7200 2400
+F 0 "U1" H 7200 2767 50  0000 C CNN
+F 1 "TL084" H 7200 2676 50  0000 C CNN
+F 2 "Package_DIP:DIP-14_W10.16mm" H 7150 2500 50  0001 C CNN
+F 3 "http://www.ti.com/lit/ds/symlink/tl081.pdf" H 7250 2600 50  0001 C CNN
+	3    7200 2400
+	1    0    0    -1
+$EndComp
+Connection ~ 6900 2500
+Wire Wire Line
+	6900 2500 6900 2700
+$Comp
+L Amplifier_Operational:TL084 U1
+U 5 1 5F1BC580
+P 1000 4900
+F 0 "U1" H 958 4946 50  0000 L CNN
+F 1 "TL084" H 958 4855 50  0000 L CNN
+F 2 "Package_DIP:DIP-14_W10.16mm" H 950 5000 50  0001 C CNN
+F 3 "http://www.ti.com/lit/ds/symlink/tl081.pdf" H 1050 5100 50  0001 C CNN
+	5    1000 4900
+	1    0    0    -1
+$EndComp
+$Comp
+L Amplifier_Operational:TL082 U2
+U 1 1 5F3DE104
+P 2500 6250
+F 0 "U2" H 2500 5883 50  0000 C CNN
+F 1 "TL082" H 2500 5974 50  0000 C CNN
+F 2 "Package_DIP:DIP-8_W10.16mm" H 2500 6250 50  0001 C CNN
+F 3 "http://www.ti.com/lit/ds/symlink/tl081.pdf" H 2500 6250 50  0001 C CNN
+	1    2500 6250
+	1    0    0    1
+$EndComp
 $EndSCHEMATC

Commit message: cambio en huellas del kikad
Parts:
- R10, R11, R12, R13, R14, R15, R16, R17, R18, R19, R20, R21, R22, R23, R24, R25, R26, R27, R3, R4, R5, R6, R7, R8, R9, RD1, RF1: footprint Resistor_SMD:R_0603_1608Metric -> Resistor_SMD:R_1206_3216Metric
- R2, R28, R29, R30, R31, R50, R51, Rs1: footprint Resistor_SMD:R_0603_1608Metric -> Resistor_SMD:R_0805_2012Metric
- U2: footprint Package_DIP:DIP-8_W10.16mm -> Package_SO:SOIC-16W-12_7.5x10.3mm_P1.27mm
- U4: footprint Package_DIP:DIP-8_W10.16mm -> Package_DIP:DIP-28_W7.62mm_Socket_LongPads
- U5: footprint Package_SO:SOIC-16_3.9x9.9mm_P1.27mm -> Package_SO:SOIC-8-1EP_3.9x4.9mm_P1.27mm_EP2.29x3mm
- Z1: footprint kicad2:DIOAD1256W56L444D203 -> Package_SO:SOIC-8-1EP_3.9x4.9mm_P1.27mm_EP2.29x3mm
