File: Kicad/Etapa_de_potencia/_autosave-Etapa_de_potencia_final.sch (KiCad schematic (older format))
At the start: 72 parts, among them J1 Conn_01x01_Male, J10 Conn_01x01_Male, J11 Conn_01x01_Male, J12 Conn_01x01_Male, J13 Conn_01x01_Male, J2 Conn_01x01_Male, J3 Conn_01x01_Male, J4 Conn_01x02_Male, J5 Conn_01x01_Male, J6 Conn_01x01_Male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

Commit message: PCB FINAL POTENCIA
Parts:
- added Cbypass1: 0.22u, Capacitor_THT:C_Disc_D5.0mm_W2.5mm_P5.00mm, symbol Device:C
Connections:
- net GND: now also Cbypass1.2
- net VD: now also Cbypass1.1
- net at R12.2, R13.1, R17.2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: no longer R14.2, R15.1, R16.2, U1.9 (-)
- net at C1.1, R12.1, Rs1.2: now also U6.19 (20); no longer U6.18 (19)
- new net: R14.2, R15.1, R16.2, U1.9 (-)
Changed lines of the file:
@@
 	2450 3150 2600 3150
 Wire Wire Line
-	2600 3150 2600 3700
-Wire Wire Line
-	2600 3700 2800 3700
-Wire Wire Line
-	2600 3700 2600 4150
-Wire Wire Line
 	2600 4150 2650 4150
-Connection ~ 2600 3700
 Wire Wire Line
 	2600 4150 2600 4500
@@
 	5650 1500 5650 1850
 Wire Wire Line
-	5650 2150 5650 2300
-Wire Wire Line
 	6100 2150 6100 2300
 Wire Wire Line
@@
 Wire Wire Line
 	6100 2300 6100 2450
-Wire Wire Line
-	6100 2300 5650 2300
-Connection ~ 5650 2300
-Wire Wire Line
-	5650 2300 5650 2400
-Wire Wire Line
-	5650 2300 5400 2300
 Wire Wire Line
 	5650 2400 6900 2400
@@
 	8850 3850 8850 3550
 Wire Wire Line
-	8850 3300 9100 3300
+	8850 3300 9050 3300
 Connection ~ 8850 3550
 Wire Wire Line
@@
 	9400 4350 9550 4350
 Wire Wire Line
-	12250 4350 12550 4350
-Wire Wire Line
 	14350 3950 14350 4750
 Wire Wire Line
 	9350 3950 14350 3950
 Wire Wire Line
-	12550 1800 12550 4350
+	12550 1800 12550 4150
 Wire Wire Line
 	6100 1800 12550 1800
@@
 Wire Wire Line
 	10500 1650 10500 1500
+Wire Wire Line
+	2600 3700 2600 4150
+Wire Wire Line
+	2600 3150 2600 3700
+Connection ~ 2600 3700
+Wire Wire Line
+	2600 3700 2800 3700
+Wire Wire Line
+	5650 2150 5650 2400
+Wire Wire Line
+	5400 2300 6100 2300
+$Comp
+L Device:C Cbypass1
+U 1 1 5F63E5DE
+P 9050 3150
+F 0 "Cbypass1" H 8935 3104 50  0000 R CNN
+F 1 "0.22u" H 8935 3195 50  0000 R CNN
+F 2 "Capacitor_THT:C_Disc_D5.0mm_W2.5mm_P5.00mm" H 9088 3000 50  0001 C CNN
+F 3 "~" H 9050 3150 50  0001 C CNN
+	1    9050 3150
+	-1   0    0    1
+$EndComp
+Connection ~ 9050 3300
+Wire Wire Line
+	9050 3300 9100 3300
+$Comp
+L power:GND #PWR04
+U 1 1 5F63F972
+P 9050 2950
+F 0 "#PWR04" H 9050 2700 50  0001 C CNN
+F 1 "GND" H 9055 2777 50  0000 C CNN
+F 2 "" H 9050 2950 50  0001 C CNN
+F 3 "" H 9050 2950 50  0001 C CNN
+	1    9050 2950
+	-1   0    0    1
+$EndComp
+Wire Wire Line
+	9050 3000 9050 2950
+Wire Wire Line
+	12250 4150 12550 4150
+Wire Wire Line
+	12550 4150 12550 4350
+Connection ~ 12550 4150
+Wire Wire Line
+	12550 4150 12550 4350
 $EndSCHEMATC
