File: Kicad/Etapa_de_potencia/Etapa_de_potencia_final.kicad_pcb (KiCad board)
At the start: 2 copper layers, 73 parts, among them J1 Conn_01x01_Male, J10 Conn_01x01_Male, J11 Conn_01x01_Male, J12 Conn_01x01_Male, J13 Conn_01x01_Male, J2 Conn_01x01_Male, J3 Conn_01x01_Male, J4 Conn_01x02_Male, J5 Conn_01x01_Male, J6 Conn_01x01_Male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

Commit message: PCB FINAL POTENCIA
Parts:
- removed L1: 2m, Inductor_THT:L_Axial_L26.7mm_D14.0mm_P35.00mm_Horizontal_Vishay_IHA-104
- removed the R20 at (70.8, 47.2)
- added Cbypass1: 22u, Capacitor_THT:C_Disc_D5.0mm_W2.5mm_P5.00mm, F.Cu at (115.6, 73.9)
- added U6: TI-ETD49-2350, TI-ETD49-2350:ETD49-K-H-20P, F.Cu at (150.4, 104.1)
- moved R12 36.7 mm to (80.8, 59.9), turned to 90 degrees
- moved D5 31.4 mm to (119.4, 69.1), turned to 180 degrees
- moved R14 29.3 mm to (84.3, 58.9), turned to 180 degrees
- moved J8 27.5 mm to (119.1, 53.8), turned to 180 degrees
- moved R23 25.2 mm to (100.6, 40.1)
- moved R21 25.0 mm to (100.6, 38.1)
- moved C8 24.2 mm to (95.5, 38.1), turned to 0 degrees
- moved C10 24.2 mm to (95.5, 40.6)
- moved R6 23.0 mm to (91.9, 39.1)
- moved Rs1 17.1 mm to (117.6, 59.9), turned to 270 degrees
- moved D3 16.7 mm to (139.2, 63.5)
- moved J7 12.3 mm to (112.3, 105.9)
- moved Q5 8.89 mm to (117.3, 95.5), turned to 270 degrees
- moved Z1 7.69 mm to (98.0, 56.4), turned to 180 degrees
- moved R13 5.14 mm to (77.0, 55.4)
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Connections:
- R14 pad 2: Net-(R12-Pad2) -> Net-(R14-Pad2)
- R15 pad 1: Net-(R12-Pad2) -> Net-(R14-Pad2)
- R16 pad 2: Net-(R12-Pad2) -> Net-(R14-Pad2)
- U1 pad 9: Net-(R12-Pad2) -> Net-(R14-Pad2)
Routing:
- net GND: track 39.9 -> 208.0 mm, vias 5 -> 6
- net VD: track 74.2 -> 129.1 mm
- net Net-(C1-Pad1): track 37.7 -> 80.5 mm
- net Net-(R12-Pad2): track 57.7 -> 17.8 mm
- net Net-(C2-Pad1): track 96.3 -> 129.8 mm
- net +5V: track 54.8 -> 83.1 mm
- net Net-(J8-Pad2): track 42.2 -> 59.0 mm
- net Net-(R14-Pad2): track 0.00 -> 15.8 mm
- net Net-(C6-Pad1): track 26.3 -> 12.6 mm
- net Net-(C10-Pad1): track 94.6 -> 81.6 mm
- net -5V: track 70.3 -> 78.5 mm, vias 0 -> 1
- net Net-(C5-Pad1): track 11.5 -> 16.9 mm
- net Net-(C11-Pad2): track 21.3 -> 17.1 mm
- net Net-(D4-Pad2): track 11.3 -> 8.48 mm
- net Net-(Q1-Pad2): track 12.6 -> 14.5 mm
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
Commit message: KICAD
Parts:
- Cbypass1: value 22u -> 1000u; footprint Capacitor_THT:C_Disc_D5.0mm_W2.5mm_P5.00mm -> Capacitor_THT:C_Radial_D16.0mm_H25.0mm_P7.50mm
- Q4, Q5: footprint IRF510:TO220 -> eec:Vishay-IRF510-0
- moved D5 28.8 mm to (123.7, 97.5), turned to 90 degrees
- moved D3 14.0 mm to (130.8, 74.7)
- moved Cbypass1 12.8 mm to (104.1, 68.1)
- moved J7 11.7 mm to (123.7, 108.2)
- moved U6 9.71 mm to (140.7, 103.1)
- moved C1 9.45 mm to (122.2, 63.0)
- moved Q5 7.18 mm to (110.2, 96.5), turned to 0 degrees
- moved Q4 6.97 mm to (110.5, 82.5), turned to 0 degrees
- moved C5 3.20 mm to (105.9, 84.2), turned to 270 degrees
Routing:
- net Net-(C2-Pad1): track 129.8 -> 96.5 mm
- net VD: track 129.1 -> 105.8 mm
- net GND: track 208.0 -> 222.7 mm
- net Net-(C1-Pad1): track 80.5 -> 67.6 mm
- net Net-(C5-Pad1): track 16.9 -> 9.49 mm
- net Net-(C6-Pad1): track 12.6 -> 11.5 mm
