File: Kicad/Etapa_de_potencia/Etapa_de_potencia_final.sch (KiCad schematic (older format))
At the start: 72 parts, among them J1 Conn_01x01_Male, J10 Conn_01x01_Male, J11 Conn_01x01_Male, J12 Conn_01x01_Male, J13 Conn_01x01_Male, J2 Conn_01x01_Male, J3 Conn_01x01_Male, J4 Conn_01x02_Male, J5 Conn_01x01_Male, J6 Conn_01x01_Male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

Commit message: PCB FINAL POTENCIA
Parts:
- removed L1: 2m, Inductor_THT:L_Axial_L26.7mm_D14.0mm_P35.00mm_Horizontal_Vishay_IHA-104, symbol Device:L
- added Cbypass1: 22u, Capacitor_THT:C_Disc_D5.0mm_W2.5mm_P5.00mm, symbol Device:C
- added U6: TI-ETD49-2350, TI-ETD49-2350:ETD49-K-H-20P, symbol TI-ETD49-2350:TI-ETD49-2350
Connections:
- net GND: now also Cbypass1.2
- net VD: now also Cbypass1.1
- net at R12.2, R13.1, R17.2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: no longer R14.2, R15.1, R16.2, U1.9 (-)
- net at C2.1, C5.2, D3.2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: now also U6.2
- net at C1.1, R12.1, Rs1.2: now also U6.18 (19)
- new net: R14.2, R15.1, R16.2, U1.9 (-)
Other:
- moved on the sheet: C1, J8, Rs1
Changed lines of the file:
@@
 	2450 3150 2600 3150
 Wire Wire Line
-	2600 3150 2600 3700
-Wire Wire Line
-	2600 3700 2800 3700
-Wire Wire Line
-	2600 3700 2600 4150
-Wire Wire Line
 	2600 4150 2650 4150
-Connection ~ 2600 3700
 Wire Wire Line
 	2600 4150 2600 4500
@@
 	5650 1500 5650 1850
 Wire Wire Line
-	5650 2150 5650 2300
-Wire Wire Line
 	6100 2150 6100 2300
 Wire Wire Line
@@
 Wire Wire Line
 	6100 2300 6100 2450
-Wire Wire Line
-	6100 2300 5650 2300
-Connection ~ 5650 2300
-Wire Wire Line
-	5650 2300 5650 2400
-Wire Wire Line
-	5650 2300 5400 2300
 Wire Wire Line
 	5650 2400 6900 2400
@@
 Wire Wire Line
 	1200 4600 1200 4750
-$Comp
-L Device:L L1
-U 1 1 5F2DA743
-P 9550 4200
-F 0 "L1" V 9740 4200 50  0000 C CNN
-F 1 "2m" V 9649 4200 50  0000 C CNN
-F 2 "Inductor_THT:L_Axial_L26.7mm_D14.0mm_P35.00mm_Horizontal_Vishay_IHA-104" H 9550 4200 50  0001 C CNN
-F 3 "~" H 9550 4200 50  0001 C CNN
-	1    9550 4200
-	0    -1   -1   0
-$EndComp
 Connection ~ 9300 4200
-Wire Wire Line
-	9300 4200 9400 4200
 Wire Wire Line
 	9350 3300 9350 3950
@@
 Connection ~ 5650 1500
 Wire Wire Line
-	11400 4600 11400 4500
-Wire Wire Line
-	11700 4600 11400 4600
-Wire Wire Line
-	11700 3950 11700 4600
-Wire Wire Line
-	9350 3950 11700 3950
-Wire Wire Line
-	11400 4400 11400 4200
+	14050 4750 14050 4650
+Wire Wire Line
+	14350 4750 14050 4750
+Wire Wire Line
+	14050 4550 14050 4350
 $Comp
 L Connector:Screw_Terminal_01x02 J8
 U 1 1 5F234C80
-P 11200 4500
-F 0 "J8" H 11118 4175 50  0000 C CNN
-F 1 "Screw_Terminal_01x02" H 11118 4266 50  0000 C CNN
-F 2 "TerminalBlock:TerminalBlock_bornier-2_P5.08mm" H 11200 4500 50  0001 C CNN
-F 3 "~" H 11200 4500 50  0001 C CNN
-	1    11200 4500
-	-1   0    0    1
-$EndComp
-Wire Wire Line
-	9900 4200 10150 4200
+P 13850 4650
+F 0 "J8" H 13768 4325 50  0000 C CNN
+F 1 "Screw_Terminal_01x02" H 13768 4416 50  0000 C CNN
+F 2 "TerminalBlock:TerminalBlock_bornier-2_P5.08mm" H 13850 4650 50  0001 C CNN
+F 3 "~" H 13850 4650 50  0001 C CNN
+	1    13850 4650
+	-1   0    0    1
+$EndComp
+Wire Wire Line
+	12550 4350 12800 4350
 $Comp
 L Device:R Rs1
 U 1 1 5F295444
-P 10300 4200
-F 0 "Rs1" V 10093 4200 50  0000 C CNN
-F 1 "0.1" V 10184 4200 50  0000 C CNN
-F 2 "Resistor_SMD:R_0603_1608Metric" V 10230 4200 50  0001 C CNN
-F 3 "~" H 10300 4200 50  0001 C CNN
-	1    10300 4200
-	0    1    1    0
-$EndComp
-Wire Wire Line
-	10450 4200 10500 4200
-Wire Wire Line
-	9900 1800 9900 4200
-Wire Wire Line
-	9900 1800 6100 1800
+P 12950 4350
+F 0 "Rs1" V 12743 4350 50  0000 C CNN
+F 1 "0.1" V 12834 4350 50  0000 C CNN
+F 2 "Resistor_SMD:R_0603_1608Metric" V 12880 4350 50  0001 C CNN
+F 3 "~" H 12950 4350 50  0001 C CNN
+	1    12950 4350
+	0    1    1    0
+$EndComp
+Wire Wire Line
+	13100 4350 13150 4350
 Wire Wire Line
 	5650 1500 10500 1500
-Connection ~ 10500 4200
-Wire Wire Line
-	10500 1500 10500 4200
+Connection ~ 13150 4350
+Wire Wire Line
+	13150 1650 13150 4350
 $Comp
 L power:GND #PWR024
 U 1 1 5F29DB3C
-P 9900 4500
-F 0 "#PWR024" H 9900 4250 50  0001 C CNN
-F 1 "GND" H 9905 4327 50  0000 C CNN
-F 2 "" H 9900 4500 50  0001 C CNN
-F 3 "" H 9900 4500 50  0001 C CNN
-	1    9900 4500
-	1    0    0    -1
-$EndComp
-Connection ~ 9900 4200
-Wire Wire Line
-	9700 4200 9900 4200
+P 12550 4650
+F 0 "#PWR024" H 12550 4400 50  0001 C CNN
+F 1 "GND" H 12555 4477 50  0000 C CNN
+F 2 "" H 12550 4650 50  0001 C CNN
+F 3 "" H 12550 4650 50  0001 C CNN
+	1    12550 4650
+	1    0    0    -1
+$EndComp
+Connection ~ 12550 4350
 $Comp
 L Device:C C1
 U 1 1 5F294A68
-P 9900 4350
-F 0 "C1" H 10015 4396 50  0000 L CNN
-F 1 "1u" H 10015 4305 50  0000 L CNN
-F 2 "Capacitor_THT:C_Radial_D5.0mm_H11.0mm_P2.00mm" H 9938 4200 50  0001 C CNN
-F 3 "~" H 9900 4350 50  0001 C CNN
-	1    9900 4350
+P 12550 4500
+F 0 "C1" H 12665 4546 50  0000 L CNN
+F 1 "1u" H 12665 4455 50  0000 L CNN
+F 2 "Capacitor_THT:C_Radial_D5.0mm_H11.0mm_P2.00mm" H 12588 4350 50  0001 C CNN
+F 3 "~" H 12550 4500 50  0001 C CNN
+	1    12550 4500
 	1    0    0    -1
 $EndComp
@@
 	8850 3850 8850 3550
 Wire Wire Line
-	8850 3300 9100 3300
+	8850 3300 9050 3300
 Connection ~ 8850 3550
 Wire Wire Line
@@
 $EndComp
 Wire Wire Line
-	10500 4200 11400 4200
+	13150 4350 14050 4350
 Connection ~ 7250 3900
 Wire Wire Line
@@
 Wire Wire Line
 	2950 4150 3000 4150
+$Comp
+L TI-ETD49-2350:TI-ETD49-2350 U6
+U 1 1 5F46A25C
+P 10250 4650
+F 0 "U6" H 10900 5417 50  0000 C CNN
+F 1 "TI-ETD49-2350" H 10900 5326 50  0000 C CNN
+F 2 "TI-ETD49-2350:ETD49-K-H-20P" H 10250 4650 50  0001 L BNN
+F 3 "" H 10250 4650 50  0001 C CNN
+	1    10250 4650
+	1    0    0    -1
+$EndComp
+Wire Wire Line
+	9300 4200 9400 4200
+Wire Wire Line
+	9400 4200 9400 4350
+Wire Wire Line
+	9400 4350 9550 4350
+Wire Wire Line
+	12250 4350 12550 4350
+Wire Wire Line
+	14350 3950 14350 4750
+Wire Wire Line
+	9350 3950 14350 3950
+Wire Wire Line
+	12550 1800 12550 4350
+Wire Wire Line
+	6100 1800 12550 1800
+Wire Wire Line
+	13150 1650 10500 1650
+Wire Wire Line
+	10500 1650 10500 1500
+Wire Wire Line
+	2600 3700 2600 4150
+Wire Wire Line
+	2600 3150 2600 3700
+Connection ~ 2600 3700
+Wire Wire Line
+	2600 3700 2800 3700
+Wire Wire Line
+	5650 2150 5650 2400
+Wire Wire Line
+	5400 2300 6100 2300
+$Comp
+L Device:C Cbypass1
+U 1 1 5F63E5DE
+P 9050 3150
+F 0 "Cbypass1" H 8935 3104 50  0000 R CNN
+F 1 "22u" H 8935 3195 50  0000 R CNN
+F 2 "Capacitor_THT:C_Disc_D5.0mm_W2.5mm_P5.00mm" H 9088 3000 50  0001 C CNN
+F 3 "~" H 9050 3150 50  0001 C CNN
+	1    9050 3150
+	-1   0    0    1
+$EndComp
+Connection ~ 9050 3300
+Wire Wire Line
+	9050 3300 9100 3300
+$Comp
+L power:GND #PWR04
+U 1 1 5F63F972
+P 9050 2950
+F 0 "#PWR04" H 9050 2700 50  0001 C CNN
+F 1 "GND" H 9055 2777 50  0000 C CNN
+F 2 "" H 9050 2950 50  0001 C CNN
+F 3 "" H 9050 2950 50  0001 C CNN
+	1    9050 2950
+	-1   0    0    1
+$EndComp
+Wire Wire Line
+	9050 3000 9050 2950
 $EndSCHEMATC

Commit message: KICAD
Parts:
- removed Q4, Q5: IRF510, IRF510:TO220, symbol IRF510:IRF510
- added Q4, Q5: IRF510, eec:Vishay-IRF510-0, symbol eec:IRF510
- Cbypass1: value 22u -> 1000u; footprint Capacitor_THT:C_Disc_D5.0mm_W2.5mm_P5.00mm -> Capacitor_THT:C_Radial_D16.0mm_H25.0mm_P7.50mm
Connections:
- net GND: now also Q5.3 (S)
- net VD: now also Q4.2 (D)
- net at C2.1, C5.2, D3.2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: now also Q4.3 (S), Q5.2 (D)
- net at C5.1, R4.1: now also Q4.1 (G)
- net at C6.1, R5.1: now also Q5.1 (G)
- net at C1.1, R12.1, Rs1.2: now also U6.19 (20); no longer U6.18 (19)
Other:
- moved on the sheet: C6
Changed lines of the file:
@@
 	1    0    0    -1
 $EndComp
-Wire Wire Line
-	8450 4750 8350 4750
-Wire Wire Line
-	8250 4750 8250 4700
-Wire Wire Line
-	8250 4700 8150 4700
 $Comp
 L power:GND #PWR020
@@
 P 9100 3600
 F 0 "D3" V 9354 3728 50  0000 L CNN
-F 1 "MUR460G" H 9200 3400 50  0000 L CNN
+F 1 "MUR460G" H 8950 3750 50  0000 L CNN
 F 2 "kicad2:DIOAD2860W130L840D505" H 9550 3600 50  0001 L CNN
 F 3 "http://www.onsemi.com/pub/Collateral/MUR420-D.PDF" H 9550 3500 50  0001 L CNN
@@
 Connection ~ 6150 7400
 Connection ~ 5300 6550
-$Comp
-L IRF510:IRF510 Q5
-U 1 1 5F5E641A
-P 8650 4650
-F 0 "Q5" H 8650 4962 50  0000 C CNN
-F 1 "IRF510" H 8650 4871 50  0000 C CNN
-F 2 "IRF510:TO220" H 8650 4650 50  0001 C CNN
-F 3 "" H 8650 4650 50  0001 C CNN
-	1    8650 4650
-	1    0    0    -1
-$EndComp
-$Comp
-L IRF510:IRF510 Q4
-U 1 1 5F5EB9CA
-P 8650 3950
-F 0 "Q4" H 8650 4262 50  0000 C CNN
-F 1 "IRF510" H 8650 4171 50  0000 C CNN
-F 2 "IRF510:TO220" H 8650 3950 50  0001 C CNN
-F 3 "" H 8650 3950 50  0001 C CNN
-	1    8650 3950
-	1    0    0    -1
-$EndComp
-Wire Wire Line
-	8850 4200 8850 4550
 Wire Wire Line
 	8850 4200 9100 4200
-Wire Wire Line
-	8850 4050 8850 4200
 Connection ~ 8850 4200
 Wire Wire Line
@@
 Wire Wire Line
 	6250 4600 7850 4600
-Wire Wire Line
-	8450 3900 8450 4050
-Wire Wire Line
-	8850 3850 8850 3550
 Wire Wire Line
 	8850 3300 9050 3300
 Connection ~ 8850 3550
-Wire Wire Line
-	8850 4750 8850 4900
 Wire Wire Line
 	2950 2550 2950 3000
@@
 Wire Wire Line
 	7250 3900 7700 3900
-Wire Wire Line
-	8450 3900 8150 3900
 $Comp
 L Device:C C5
@@
 L Device:C C6
 U 1 1 5F7018ED
-P 8350 4900
-F 0 "C6" H 8465 4946 50  0000 L CNN
-F 1 "1n" H 8465 4855 50  0000 L CNN
-F 2 "Capacitor_SMD:C_1206_3216Metric" H 8388 4750 50  0001 C CNN
-F 3 "~" H 8350 4900 50  0001 C CNN
-	1    8350 4900
-	1    0    0    -1
-$EndComp
-Connection ~ 8350 4750
-Wire Wire Line
-	8350 4750 8250 4750
+P 8350 4850
+F 0 "C6" H 8465 4896 50  0000 L CNN
+F 1 "1n" H 8465 4805 50  0000 L CNN
+F 2 "Capacitor_SMD:C_1206_3216Metric" H 8388 4700 50  0001 C CNN
+F 3 "~" H 8350 4850 50  0001 C CNN
+	1    8350 4850
+	1    0    0    -1
+$EndComp
+Connection ~ 8350 4700
 $Comp
 L power:GND #PWR03
 U 1 1 5F701D49
-P 8350 5050
-F 0 "#PWR03" H 8350 4800 50  0001 C CNN
-F 1 "GND" V 8355 4922 50  0000 R CNN
-F 2 "" H 8350 5050 50  0001 C CNN
-F 3 "" H 8350 5050 50  0001 C CNN
-	1    8350 5050
+P 8350 5000
+F 0 "#PWR03" H 8350 4750 50  0001 C CNN
+F 1 "GND" V 8355 4872 50  0000 R CNN
+F 2 "" H 8350 5000 50  0001 C CNN
+F 3 "" H 8350 5000 50  0001 C CNN
+	1    8350 5000
 	1    0    0    -1
 $EndComp
@@
 	9400 4350 9550 4350
 Wire Wire Line
-	12250 4350 12550 4350
-Wire Wire Line
 	14350 3950 14350 4750
 Wire Wire Line
 	9350 3950 14350 3950
 Wire Wire Line
-	12550 1800 12550 4350
+	12550 1800 12550 4150
 Wire Wire Line
 	6100 1800 12550 1800
@@
 P 9050 3150
 F 0 "Cbypass1" H 8935 3104 50  0000 R CNN
-F 1 "22u" H 8935 3195 50  0000 R CNN
-F 2 "Capacitor_THT:C_Disc_D5.0mm_W2.5mm_P5.00mm" H 9088 3000 50  0001 C CNN
+F 1 "1000u" H 8935 3195 50  0000 R CNN
+F 2 "Capacitor_THT:C_Radial_D16.0mm_H25.0mm_P7.50mm" H 9088 3000 50  0001 C CNN
 F 3 "~" H 9050 3150 50  0001 C CNN
 	1    9050 3150
@@
 Wire Wire Line
 	9050 3000 9050 2950
+Wire Wire Line
+	12250 4150 12550 4150
+Wire Wire Line
+	12550 4150 12550 4350
+Connection ~ 12550 4150
+$Comp
+L eec:IRF510 Q4
+U 1 1 5F68036E
+P 8450 3900
+F 0 "Q4" H 8894 3946 50  0000 L CNN
+F 1 "IRF510" H 8894 3855 50  0000 L CNN
+F 2 "eec:Vishay-IRF510-0" H 8450 4400 50  0001 L CNN
+F 3 "http://www.vishay.com/docs/91015/sihf510.pdf" H 8450 4500 50  0001 L CNN
+F 4 "Trans" H 8450 4600 50  0001 L CNN "category"
+F 5 "MOSFET N-CH 100V 5.6A TO-220AB" H 8450 4700 50  0001 L CNN "digikey description"
+F 6 "IRF510-ND" H 8450 4800 50  0001 L CNN "digikey part number"
+F 7 "TO-220" H 8450 4900 50  0001 L CNN "ipc land pattern name"
+F 8 "Yes" H 8450 5000 50  0001 L CNN "lead free"
+F 9 "f36e9f9f8fc5fc57" H 8450 5100 50  0001 L CNN "library id"
+F 10 "Vishay" H 8450 5200 50  0001 L CNN "manufacturer"
+F 11 "844-IRF510" H 8450 5300 50  0001 L CNN "mouser part number"
+F 12 "TO-263-3" H 8450 5400 50  0001 L CNN "package"
+F 13 "Yes" H 8450 5500 50  0001 L CNN "rohs"
+F 14 "+175°C" H 8450 5600 50  0001 L CNN "temperature range high"
+F 15 "-55°C" H 8450 5700 50  0001 L CNN "temperature range low"
+	1    8450 3900
+	1    0    0    -1
+$EndComp
+Wire Wire Line
+	8850 4100 8850 4200
+Wire Wire Line
+	8850 3700 8850 3550
+$Comp
+L eec:IRF510 Q5
+U 1 1 5F68378A
+P 8450 4700
+F 0 "Q5" H 8894 4746 50  0000 L CNN
+F 1 "IRF510" H 8894 4655 50  0000 L CNN
+F 2 "eec:Vishay-IRF510-0" H 8450 5200 50  0001 L CNN
+F 3 "http://www.vishay.com/docs/91015/sihf510.pdf" H 8450 5300 50  0001 L CNN
+F 4 "Trans" H 8450 5400 50  0001 L CNN "category"
+F 5 "MOSFET N-CH 100V 5.6A TO-220AB" H 8450 5500 50  0001 L CNN "digikey description"
+F 6 "IRF510-ND" H 8450 5600 50  0001 L CNN "digikey part number"
+F 7 "TO-220" H 8450 5700 50  0001 L CNN "ipc land pattern name"
+F 8 "Yes" H 8450 5800 50  0001 L CNN "lead free"
+F 9 "f36e9f9f8fc5fc57" H 8450 5900 50  0001 L CNN "library id"
+F 10 "Vishay" H 8450 6000 50  0001 L CNN "manufacturer"
+F 11 "844-IRF510" H 8450 6100 50  0001 L CNN "mouser part number"
+F 12 "TO-263-3" H 8450 6200 50  0001 L CNN "package"
+F 13 "Yes" H 8450 6300 50  0001 L CNN "rohs"
+F 14 "+175°C" H 8450 6400 50  0001 L CNN "temperature range high"
+F 15 "-55°C" H 8450 6500 50  0001 L CNN "temperature range low"
+	1    8450 4700
+	1    0    0    -1
+$EndComp
+Wire Wire Line
+	8850 4500 8850 4200
+Wire Wire Line
+	8350 4700 8550 4700
+Wire Wire Line
+	8150 4700 8350 4700
+Wire Wire Line
+	8150 3900 8550 3900
 $EndSCHEMATC
