File: kikad2022/Proyecto_completo/Control2.sch (KiCad schematic (older format))
At the start: 22 parts, among them Q22 Q_PMOS_DGS, U10 TL084, U9 TL084

Commit message: kikad_modificaciones
Parts:
- added unit 5 of U10
Connections:
- net -5V: now also U9.11 (V-), U10.11 (V-)
- net +15V: now reaches U9.4 (V+)
- net +15V: now also U10.4 (V+)
Changed lines of the file:
@@
 	1    0    0    -1
 $EndComp
+$Comp
+L power:-5V #PWR035
+U 1 1 6274420C
+P 2800 2500
+F 0 "#PWR035" H 2800 2600 50  0001 C CNN
+F 1 "-5V" H 2815 2673 50  0000 C CNN
+F 2 "" H 2800 2500 50  0001 C CNN
+F 3 "" H 2800 2500 50  0001 C CNN
+	1    2800 2500
+	-1   0    0    1
+$EndComp
+$Comp
+L Amplifier_Operational:TL084 U10
+U 5 1 62744A2E
+P 3150 2250
+F 0 "U10" H 3150 1883 50  0000 C CNN
+F 1 "TL084" H 3150 1974 50  0000 C CNN
+F 2 "New folder:SOIC127P600X175-14N" H 3100 2350 50  0001 C CNN
+F 3 "http://www.ti.com/lit/ds/symlink/tl081.pdf" H 3200 2450 50  0001 C CNN
+	5    3150 2250
+	-1   0    0    -1
+$EndComp
+$Comp
+L power:+15V #PWR045
+U 1 1 62749A5C
+P 3250 1950
+F 0 "#PWR045" H 3250 1800 50  0001 C CNN
+F 1 "+15V" H 3265 2123 50  0000 C CNN
+F 2 "" H 3250 1950 50  0001 C CNN
+F 3 "" H 3250 1950 50  0001 C CNN
+	1    3250 1950
+	1    0    0    -1
+$EndComp
+$Comp
+L power:+15V #PWR029
+U 1 1 6274A129
+P 2800 1900
+F 0 "#PWR029" H 2800 1750 50  0001 C CNN
+F 1 "+15V" H 2815 2073 50  0000 C CNN
+F 2 "" H 2800 1900 50  0001 C CNN
+F 3 "" H 2800 1900 50  0001 C CNN
+	1    2800 1900
+	1    0    0    -1
+$EndComp
+$Comp
+L power:-5V #PWR049
+U 1 1 6274A5A3
+P 3250 2550
+F 0 "#PWR049" H 3250 2650 50  0001 C CNN
+F 1 "-5V" H 3265 2723 50  0000 C CNN
+F 2 "" H 3250 2550 50  0001 C CNN
+F 3 "" H 3250 2550 50  0001 C CNN
+	1    3250 2550
+	-1   0    0    1
+$EndComp
 $EndSCHEMATC
